Commit message: Added Correct Files

File: mybot_description/urdf/umic.xacro (robot description, xacro)
@@ -1,7 +1,7 @@
 <?xml version='1.0'?>
 <robot name="myrobot" xmlns:xacro="http://www.ros.org/wiki/xacro">
-  <xacro:include filename="$(find mybot_description)/urdf/mybot.gazebo" />
+  <xacro:include filename="$(find mybot_description)/urdf/umic.gazebo" />
   <xacro:include filename="$(find mybot_description)/urdf/materials.xacro" />
-  <xacro:include filename="$(find mybot_description)/urdf/macros.xacro" />
+  <!--xacro:include filename="$(find mybot_description)/urdf/macros.xacro" /-->
   <link name='chassis'>
     <pose>0 0 0.1 0 0 0</pose>
@@ -27,7 +27,7 @@
     </visual>
   </link>
-  <link name="left_front_wheel">
+  <!--link name="left_front_wheel"-->
     <!--origin xyz="0.1 0.13 0.1" rpy="0 1.5707 1.5707"/-->
-    <collision name="collision">
+    <!--collision name="collision">
       <origin xyz="0 0 0" rpy="0 1.5707 1.5707"/>
       <geometry>
@@ -50,11 +50,11 @@
         izz="1.0"/>
     </inertial>
-  </link>
-  <link name="left_back_wheel">
+  </link-->
+  <link name="left_wheel">
     <!--origin xyz="0.1 0.13 0.1" rpy="0 1.5707 1.5707"/-->
     <collision name="collision">
       <origin xyz="0 0 0" rpy="0 1.5707 1.5707"/>
       <geometry>
-        <cylinder radius="0.07" length="0.07"/>
+        <cylinder radius="0.1" length="0.07"/>
       </geometry>
     </collision>
@@ -62,5 +62,5 @@
       <origin xyz="0 0 0" rpy="0 1.5707 1.5707"/>
       <geometry>
-        <cylinder radius="0.07" length="0.07"/>
+        <cylinder radius="0.1" length="0.07"/>
       </geometry>
     </visual>
@@ -75,10 +75,10 @@
     </inertial>
   </link>
-  <link name="right_front_wheel">
+  <link name="front_wheel">
     <!--origin xyz="0.1 -0.13 0.1" rpy="0 1.5707 1.5707"/-->
     <collision name="collision">
       <origin xyz="0 0 0" rpy="0 1.5707 1.5707"/>
       <geometry>
-        <cylinder radius="0.07" length="0.07"/>
+        <cylinder radius="0.1" length="0.07"/>
       </geometry>
     </collision>
@@ -86,5 +86,5 @@
       <origin xyz="0 0 0" rpy="0 1.5707 1.5707"/>
       <geometry>
-        <cylinder radius="0.07" length="0.07"/>
+        <cylinder radius="0.1" length="0.07"/>
       </geometry>
     </visual>
@@ -99,10 +99,10 @@
     </inertial>
   </link>
-  <link name="right_back_wheel">
+  <link name="right_wheel">
     <!--origin xyz="0.1 -0.13 0.1" rpy="0 1.5707 1.5707"/-->
     <collision name="collision">
       <origin xyz="0 0 0" rpy="0 1.5707 1.5707"/>
       <geometry>
-        <cylinder radius="0.07" length="0.05"/>
+        <cylinder radius="0.1" length="0.05"/>
       </geometry>
     </collision>
@@ -110,5 +110,5 @@
       <origin xyz="0 0 0" rpy="0 1.5707 1.5707"/>
       <geometry>
-        <cylinder radius="0.07" length="0.07"/>
+        <cylinder radius="0.1" length="0.07"/>
       </geometry>
     </visual>
@@ -123,7 +123,7 @@
     </inertial>
   </link>
-  <joint type="continuous" name="left_front_wheel_hinge">
-    <origin xyz="0.15 0.15 -0.2" rpy="0 0 0"/>
-    <child link="left_front_wheel"/>
+  <joint type="continuous" name="left_wheel_hinge">
+    <origin xyz="-0.15 0.22 -0.2" rpy="0 0 0"/>
+    <child link="right_wheel"/>
     <parent link="chassis"/>
     <axis xyz="0 1 0" rpy="0 0 0"/>
@@ -131,7 +131,7 @@
     <joint_properties damping="0.0" friction="0.0"/>
   </joint>
-  <joint type="continuous" name="left_back_wheel_hinge">
-    <origin xyz="-0.15 0.15 -0.2" rpy="0 0 0"/>
-    <child link="left_back_wheel"/>
+  <joint type="continuous" name="right_wheel_hinge">
+    <origin xyz="-0.15 -0.22 -0.2" rpy="0 0 0"/>
+    <child link="left_wheel"/>
     <parent link="chassis"/>
     <axis xyz="0 1 0" rpy="0 0 0"/>
@@ -139,7 +139,7 @@
     <joint_properties damping="0.0" friction="0.0"/>
   </joint>
-  <joint type="continuous" name="right_front_wheel_hinge">
-    <origin xyz="0.15 -0.15 -0.2" rpy="0 0 0"/>
-    <child link="right_front_wheel"/>
+  <joint type="continuous" name="front_hinge">
+    <origin xyz="0.2 0 -0.2" rpy="0 0 0"/>
+    <child link="front_wheel"/>
     <parent link="chassis"/>
     <axis xyz="0 1 0" rpy="0 0 0"/>
@@ -147,5 +147,5 @@
     <joint_properties damping="0.0" friction="0.0"/>
   </joint>
-  <joint type="continuous" name="right_back_wheel_hinge">
+  <!--joint type="continuous" name="right_back_wheel_hinge">
     <origin xyz="-0.15 -0.15 -0.2" rpy="0 0 0"/>
     <child link="right_back_wheel"/>
@@ -154,4 +154,4 @@
     <limit effort="100" velocity="100"/>
     <joint_properties damping="0.0" friction="0.0"/>
-  </joint>
+  </joint-->
 </robot>

Commit message: Changes

File: mybot_description/urdf/umic.xacro (robot description, xacro)
@@ -75,5 +75,29 @@
     </inertial>
   </link>
-  <link name="front_wheel">
+  <link name="back_left_wheel">
+    <!--origin xyz="0.1 -0.13 0.1" rpy="0 1.5707 1.5707"/-->
+    <collision name="collision">
+      <origin xyz="0 0 0" rpy="0 1.5707 1.5707"/>
+      <geometry>
+        <cylinder radius="0.1" length="0.07"/>
+      </geometry>
+    </collision>
+    <visual name="right_wheel_visual">
+      <origin xyz="0 0 0" rpy="0 1.5707 1.5707"/>
+      <geometry>
+        <cylinder radius="0.1" length="0.07"/>
+      </geometry>
+    </visual>
+    <inertial>
+      <origin xyz="0 0 0" rpy="0 1.5707 1.5707"/>
+      <mass value="5"/>
+      <cylinder_inertia m="5" r="0.1" h="0.05"/>
+      <inertia
+        ixx="1.0" ixy="0.0" ixz="0.0"
+        iyy="1.0" iyz="0.0"
+        izz="1.0"/>
+    </inertial>
+  </link>
+<link name="back_right_wheel">
     <!--origin xyz="0.1 -0.13 0.1" rpy="0 1.5707 1.5707"/-->
     <collision name="collision">
@@ -124,5 +148,5 @@
   </link>
   <joint type="continuous" name="left_wheel_hinge">
-    <origin xyz="-0.15 0.22 -0.2" rpy="0 0 0"/>
+    <origin xyz="0.15 0.22 -0.2" rpy="0 0 0"/>
     <child link="right_wheel"/>
     <parent link="chassis"/>
@@ -132,5 +156,5 @@
   </joint>
   <joint type="continuous" name="right_wheel_hinge">
-    <origin xyz="-0.15 -0.22 -0.2" rpy="0 0 0"/>
+    <origin xyz="0.15 -0.22 -0.2" rpy="0 0 0"/>
     <child link="left_wheel"/>
     <parent link="chassis"/>
@@ -139,7 +163,15 @@
     <joint_properties damping="0.0" friction="0.0"/>
   </joint>
-  <joint type="continuous" name="front_hinge">
-    <origin xyz="0.2 0 -0.2" rpy="0 0 0"/>
-    <child link="front_wheel"/>
+  <joint type="continuous" name="back_left_hinge">
+    <origin xyz="-0.15 0.22 -0.2" rpy="0 0 0"/>
+    <child link="back_left_wheel"/>
+    <parent link="chassis"/>
+    <axis xyz="0 1 0" rpy="0 0 0"/>
+    <limit effort="100" velocity="100"/>
+    <joint_properties damping="0.0" friction="0.0"/>
+  </joint>
+<joint type="continuous" name="back_right_hinge">
+    <origin xyz="-0.15 -0.22 -0.2" rpy="0 0 0"/>
+    <child link="back_right_wheel"/>
     <parent link="chassis"/>
     <axis xyz="0 1 0" rpy="0 0 0"/>

Commit message: Sensors Added

File: mybot_description/urdf/umic.xacro (robot description, xacro)
@@ -1,4 +1,6 @@
 <?xml version='1.0'?>
 <robot name="myrobot" xmlns:xacro="http://www.ros.org/wiki/xacro">
+  <xacro:property name="cameraSize" value="0.05"/>
+  <xacro:property name="cameraMass" value="0.1"/>
   <xacro:include filename="$(find mybot_description)/urdf/umic.gazebo" />
   <xacro:include filename="$(find mybot_description)/urdf/materials.xacro" />
@@ -187,3 +189,145 @@
     <joint_properties damping="0.0" friction="0.0"/>
   </joint-->
+ <link name="camera">
+    <collision>
+      <origin xyz="0 0 0" rpy="0 0 0"/>
+      <geometry>
+        <box size="${cameraSize} ${cameraSize} ${cameraSize}"/>
+      </geometry>
+    </collision>
+    <visual>
+      <origin xyz="0 0 0" rpy="0 0 0"/>
+      <geometry>
+        <box size="${cameraSize} ${cameraSize} ${cameraSize}"/>
+      </geometry>
+      <material name="green"/>
+    </visual>
+    <inertial>
+      <mass value="${cameraMass}" />
+      <origin xyz="0 0 0" rpy="0 0 0"/>
+      <box_inertia m="${cameraMass}" x="${cameraSize}" y="${cameraSize}" z="${cameraSize}" />
+      <inertia ixx="1e-6" ixy="0" ixz="0" iyy="1e-6" iyz="0" izz="1e-6" />
+    </inertial>
+  </link>
+  <joint name="camera_joint" type="fixed">
+    <axis xyz="0 1 0" />
+    <origin xyz=".2 0 0" rpy="0 0 0"/>
+    <parent link="chassis"/>
+    <child link="camera"/>
+  </joint>
+<joint name="ir_front_joint_1" type="fixed">
+    <axis xyz="0 1 0" />
+    <origin rpy="0 0.39269908169  0.39269908169 " xyz="0.2 0.2 -0.1" />
+    <parent link="chassis"/>
+    <child link="base_ir_front_1"/>
+</joint>
+<link name="base_ir_front_1">
+    <collision>
+      <origin xyz="0 0 0" rpy="0 0 0"/>
+      <geometry>
+        <box size="0.01 0.01 0.01"/>
+      </geometry>
+    </collision>    <visual>
+      <origin xyz="0 0 0" rpy="0 0 0"/>
+      <geometry>
+        <box size="0.01 0.01 0.01"/>
+      </geometry>
+    </visual>    <inertial>
+      <mass value="1e-5" />
+      <origin xyz="0 0 0" rpy="0 0 0"/>
+      <inertia ixx="1e-6" ixy="0" ixz="0" iyy="1e-6" iyz="0"      izz="1e-6" />
+    </inertial>
+</link>
+<joint name="ir_front_joint_2" type="fixed">
+    <axis xyz="0 1 0" />
+    <origin rpy="0 0.39269908169  -0.39269908169 " xyz="0.2 -0.2 -0.1" />
+    <parent link="chassis"/>
+    <child link="base_ir_front_2"/>
+</joint>
+<link name="base_ir_front_2">
+    <collision>
+      <origin xyz="0 0 0" rpy="0 0 0"/>
+      <geometry>
+        <box size="0.01 0.01 0.01"/>
+      </geometry>
+    </collision>    <visual>
+      <origin xyz="0 0 0" rpy="0 0 0"/>
+      <geometry>
+        <box size="0.01 0.01 0.01"/>
+      </geometry>
+    </visual>    <inertial>
+      <mass value="1e-5" />
+      <origin xyz="0 0 0" rpy="0 0 0"/>
+      <inertia ixx="1e-6" ixy="0" ixz="0" iyy="1e-6" iyz="0"      izz="1e-6" />
+    </inertial>
+</link>
+<joint name="sonar_front_joint_1" type="fixed">
+    <axis xyz="0 1 0" />
+    <origin rpy="0 0 0" xyz="0.2 0 0.1" />
+    <parent link="chassis"/>
+    <child link="base_sonar_front_1"/>
+</joint>
+<link name="base_sonar_front_1">
+    <collision>
+      <origin xyz="0 0 0" rpy="0 0 0"/>
+      <geometry>
+        <box size="0.01 0.01 0.01"/>
+      </geometry>
+    </collision>    <visual>
+      <origin xyz="0 0 0" rpy="0 0 0"/>
+      <geometry>
+        <box size="0.01 0.01 0.01"/>
+      </geometry>
+    </visual>    <inertial>
+      <mass value="1e-5" />
+      <origin xyz="0 0 0" rpy="0 0 0"/>
+      <inertia ixx="1e-6" ixy="0" ixz="0" iyy="1e-6" iyz="0" izz="1e-6" />
+    </inertial>
+ </link>
+<joint name="sonar_front_joint_2" type="fixed">
+    <axis xyz="0 1 0" />
+    <origin rpy="0 0 0" xyz="0.2 -0.19 0.1" />
+    <parent link="chassis"/>
+    <child link="base_sonar_front_2"/>
+</joint>
+<link name="base_sonar_front_2">
+    <collision>
+      <origin xyz="0 0 0" rpy="0 0 0"/>
+      <geometry>
+        <box size="0.01 0.01 0.01"/>
+      </geometry>
+    </collision>    <visual>
+      <origin xyz="0 0 0" rpy="0 0 0"/>
+      <geometry>
+        <box size="0.01 0.01 0.01"/>
+      </geometry>
+    </visual>    <inertial>
+      <mass value="1e-5" />
+      <origin xyz="0 0 0" rpy="0 0 0"/>
+      <inertia ixx="1e-6" ixy="0" ixz="0" iyy="1e-6" iyz="0" izz="1e-6" />
+    </inertial>
+ </link>
+<joint name="sonar_front_joint_3" type="fixed">
+    <axis xyz="0 1 0" />
+    <origin rpy="0 0 0" xyz="0.2 0.19 0.1" />
+    <parent link="chassis"/>
+    <child link="base_sonar_front_3"/>
+</joint>
+<link name="base_sonar_front_3">
+    <collision>
+      <origin xyz="0 0 0" rpy="0 0 0"/>
+      <geometry>
+        <box size="0.01 0.01 0.01"/>
+      </geometry>
+    </collision>    <visual>
+      <origin xyz="0 0 0" rpy="0 0 0"/>
+      <geometry>
+        <box size="0.01 0.01 0.01"/>
+      </geometry>
+    </visual>    <inertial>
+      <mass value="1e-5" />
+      <origin xyz="0 0 0" rpy="0 0 0"/>
+      <inertia ixx="1e-6" ixy="0" ixz="0" iyy="1e-6" iyz="0" izz="1e-6" />
+    </inertial>
+ </link>
 </robot>
